File: IR_Sensor.kicad_pcb (KiCad board)
At the start: 2 copper layers, 40.9 x 19 mm, 10 parts, among them J1 Conn_01x03_Pin, U1 LM358

Commit message: updated the new logo
Parts:
- removed the G*** at (187.8, 102.1)
- added G***: LOGO, logo_Footprints:imt_new3, B.Cu at (186.8, 102.4)
